File: HIDtaiko_connector_ver1.2/pcb/hidtaiko.kicad_pcb (KiCad board)
At the start: 2 copper layers, 84 x 50 mm, 19 parts, among them J2 Conn_02x05

Commit message: connector case sketch
Other:
- board text added: "＋"
- board text added: "－"
Changed lines of the file:
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@@
       (drillshape 0)
       (scaleselection 1)
-      (outputdirectory "../../../../../Desktop/hid taiko v1.2new/")
+      (outputdirectory "../../../../../Downloads/pcbpcb/")
     )
   )
@@
     (effects (font (size 2 2) (thickness 0.2)) (justify left bottom))
   )
+  (gr_text "－" (at 151.4 66.1) (layer "F.SilkS")
+    (effects (font (size 1.5 1.5) (thickness 0.3) bold) (justify left bottom))
+  )
   (gr_text "ver.1.2" (at 158 109.5) (layer "F.SilkS")
     (effects (font (face "ＭＳ Ｐ明朝") (size 4 4) (thickness 1) bold) (justify left bottom))
@@
     )
   )
+  (gr_text "＋" (at 151.4 63.5) (layer "F.SilkS")
+    (effects (font (size 1.5 1.5) (thickness 0.3) bold) (justify left bottom))
+  )
   (gr_text "PC-SW" (at 105.5 108.5) (layer "F.SilkS")
