File: HIDtaiko_connector_ver1.3/Printed board1.3/hidtaiko ver1.3.kicad_pcb (KiCad board)
At the start: 2 copper layers, 78.9 x 47.8 mm, 18 parts, among them J1 Conn_01x02_Pin, J2 Conn_01x02_Pin, J2 Conn_02x05, J3 Conn_01x02_Pin, J4 Conn_01x02_Pin, SW1 SW_PUSH, SW4 SW_PUSH, SW5 SW_PUSH, SW6 SW_PUSH, SW7 swpc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

Commit message: ino and kicad file changes
Parts:
- SW1, SW4, SW5, SW6: footprint keyboard:Kailh_Choc_V1 -> Library 自作:Redragon smd rgb mx
Routing:
- net Net-(U1-D7/6): track 67.2 -> 78.9 mm
- net Net-(U1-E6/7): track 63.0 -> 72.0 mm
- net Net-(U1-B4/8): track 53.0 -> 61.9 mm
- net Net-(J4-Pin_1): track 49.0 -> 55.8 mm
- net Net-(U1-B5/9): track 30.9 -> 26.9 mm
