File: HIDtaiko_connector_ver1.3/Printed board1.3/hidtaiko ver1.3.kicad_sch (KiCad schematic)
At the start: 14 parts, among them J1 Conn_01x02_Pin, J2 Conn_01x02_Pin, J3 Conn_01x02_Pin, J4 Conn_01x02_Pin, SW1 SW_PUSH, SW4 SW_PUSH, SW5 SW_PUSH, SW6 SW_PUSH, SW7 swpc, U1 ProMicro

Commit message: ino and kicad file changes
Parts:
- SW1, SW4, SW5, SW6: footprint keyboard:Kailh_Choc_V1 -> Library 自作:Redragon smd rgb mx
Changed lines of the file:
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@@
       (effects (font (size 1.27 1.27)))
     )
-    (property "Footprint" "keyboard:Kailh_Choc_V1" (at 69.85 106.68 0)
+    (property "Footprint" "Library 自作:Redragon smd rgb mx" (at 69.85 106.68 0)
       (effects (font (size 1.27 1.27)) hide)
     )
@@
       (effects (font (size 1.27 1.27)))
     )
-    (property "Footprint" "keyboard:Kailh_Choc_V1" (at 69.85 115.57 0)
+    (property "Footprint" "Library 自作:Redragon smd rgb mx" (at 69.85 115.57 0)
       (effects (font (size 1.27 1.27)) hide)
     )
@@
       (effects (font (size 1.27 1.27)))
     )
-    (property "Footprint" "keyboard:Kailh_Choc_V1" (at 69.85 97.79 0)
+    (property "Footprint" "Library 自作:Redragon smd rgb mx" (at 69.85 97.79 0)
       (effects (font (size 1.27 1.27)) hide)
     )
@@
       (effects (font (size 1.27 1.27)))
     )
-    (property "Footprint" "keyboard:Kailh_Choc_V1" (at 69.85 121.92 0)
+    (property "Footprint" "Library 自作:Redragon smd rgb mx" (at 69.85 121.92 0)
       (effects (font (size 1.27 1.27)) hide)
     )
